Commit message: added some parameters to the YAML, progress on xacro

File: urdf/ddrive.urdf.xacro (robot description, xacro)
@@ -1,13 +1,13 @@
 <?xml version="1.0"?>
-<robot xmlns:xacro="http://wiki.ros.org/wiki/xacro" name="twoarm">
-    <xacro:property name="props_arm" value="$(find homework2)/config/arm.yaml"/>
-    <xacro:property name="arm" value="${load_yaml(props_arm)}"/>
-    <xacro:property name="L1" value="${arm['L1']}"/>
-    <xacro:property name="L2" value="${arm['L2']}"/>
-    <xacro:property name="R1" value="${arm['R1']}"/>
-    <xacro:property name="R2" value="${arm['R2']}"/>
+<robot xmlns:xacro="http://wiki.ros.org/wiki/xacro" name="ddrive">
+    <xacro:property name="ddrive" value="$(find homework3)/config/ddrive.yaml"/>
+    <xacro:property name="ddrive" value="${load_yaml(ddrive)}"/>
+    <xacro:property name="wheelW" value="${ddrive['wheelWidth']}"/>
+    <xacro:property name="wheelR" value="${ddrive['wheelRadius']}"/>
+    <xacro:property name="L" value="${ddrive['L']}"/>
+    <xacro:property name="W" value="${ddrive['W']}"/>
+    <xacro:property name="H" value="${ddrive['H']}"/>
     <xacro:property name='pi' value="3.14159"/>
-    <link name="base_link"/>
-    <link name="arm1">
+    <link name="leftWheel">
         <inertial>
             <origin xyz="0 0 0" rpy="0 0 0" />
@@ -18,5 +18,5 @@
             <origin xyz="${L1/2} 0 0" rpy="${pi/2} 0 ${pi/2}" />
             <geometry>
-                <cylinder radius="${R1}" length="${L1}" />
+                <cylinder radius="${wheelR}" length="${wheelW}" />
             </geometry>
             <material name="blue_mat">
@@ -27,9 +27,9 @@
             <origin xyz="0 0 0" rpy="0 0 0"/>
             <geometry>
-                <cylinder radius="${R1}" length="${L1}"/>
+                <cylinder radius="${wheelR}" length="${wheelW}" />
             </geometry>
         </collision>
     </link>
-    <link name="arm2">
+    <link name="rightWheel">
         <inertial>
             <origin xyz="0 0 0" rpy="0 0 0" />
@@ -40,5 +40,5 @@
             <origin xyz="${L2/2} 0 0" rpy="${pi/2} 0 ${pi/2}" />
             <geometry>
-                <cylinder radius="${R2}" length="${L2}" />
+                <cylinder radius="${wheelR}" length="${wheelW}" />
             </geometry>
             <material name="red_mat">
@@ -49,9 +49,31 @@
             <origin xyz="0 0 0" rpy="0 0 0"/>
             <geometry>
-                <cylinder radius="${R2}" length="${L2}"/>
+                <cylinder radius="${wheelR}" length="${wheelW}" />
             </geometry>
         </collision>
     </link>
-    <link name="end_effector"/>
+    <link name="body">
+        <inertial>
+            <origin xyz="0 0 0" rpy="0 0 0" />
+            <mass value="1"/>
+            <inertia ixx="${(L2*L2/12) + (R2*R2/4)}"  ixy="0"  ixz="0" iyy="${(L2*L2/12) + (R2*R2/4)}" iyz="0" izz="${(R2*R2/2)}" />
+        </inertial>
+        <visual>
+            <origin xyz="${L2/2} 0 0" rpy="${pi/2} 0 ${pi/2}" />
+            <geometry>
+                <box size="${L} ${W} ${H}"/>
+            </geometry>
+            <material name="red_mat">
+                <color rgba="1 0 0 1" />
+            </material>
+        </visual>
+x
+        <collision>
+            <origin xyz="0 0 0" rpy="0 0 0"/>
+            <geometry>
+                <box size="${L} ${W} ${H}"/>
+            </geometry>
+        </collision>
+    </link>
     <joint name="joint1" type="continuous">
         <parent link="base_link" />

Commit message: edited some xacro parameters, added some parameters to the yaml

File: urdf/ddrive.urdf.xacro (robot description, xacro)
@@ -10,11 +10,11 @@
     <xacro:property name='pi' value="3.14159"/>
     <link name="leftWheel">
-        <inertial>
+        <!-- <inertial>
             <origin xyz="0 0 0" rpy="0 0 0" />
             <mass value="1"/>
             <inertia ixx="${(L1*L1/12) + (R1*R1/4)}"  ixy="0"  ixz="0" iyy="${(L1*L1/12) + (R1*R1/4)}" iyz="0" izz="${(R1*R1/2)}" />
-        </inertial>
+        </inertial> -->
         <visual>
-            <origin xyz="${L1/2} 0 0" rpy="${pi/2} 0 ${pi/2}" />
+            <origin xyz="${-W/2} ${-L/2} ${-H/2}" rpy="${pi/2} 0 ${pi/2}" />
             <geometry>
                 <cylinder radius="${wheelR}" length="${wheelW}" />
@@ -24,19 +24,19 @@
             </material>
         </visual>
-        <collision>
+        <!-- <collision>
             <origin xyz="0 0 0" rpy="0 0 0"/>
             <geometry>
                 <cylinder radius="${wheelR}" length="${wheelW}" />
             </geometry>
-        </collision>
+        </collision> -->
     </link>
     <link name="rightWheel">
-        <inertial>
+        <!-- <inertial>
             <origin xyz="0 0 0" rpy="0 0 0" />
             <mass value="1"/>
             <inertia ixx="${(L2*L2/12) + (R2*R2/4)}"  ixy="0"  ixz="0" iyy="${(L2*L2/12) + (R2*R2/4)}" iyz="0" izz="${(R2*R2/2)}" />
-        </inertial>
+        </inertial> -->
         <visual>
-            <origin xyz="${L2/2} 0 0" rpy="${pi/2} 0 ${pi/2}" />
+            <origin xyz="${W/2} ${L/2} ${H/2}" rpy="${pi/2} 0 ${pi/2}" />
             <geometry>
                 <cylinder radius="${wheelR}" length="${wheelW}" />
@@ -46,19 +46,19 @@
             </material>
         </visual>
-        <collision>
+        <!-- <collision>
             <origin xyz="0 0 0" rpy="0 0 0"/>
             <geometry>
                 <cylinder radius="${wheelR}" length="${wheelW}" />
             </geometry>
-        </collision>
+        </collision> -->
     </link>
     <link name="body">
-        <inertial>
+        <!-- <inertial>
             <origin xyz="0 0 0" rpy="0 0 0" />
             <mass value="1"/>
             <inertia ixx="${(L2*L2/12) + (R2*R2/4)}"  ixy="0"  ixz="0" iyy="${(L2*L2/12) + (R2*R2/4)}" iyz="0" izz="${(R2*R2/2)}" />
-        </inertial>
+        </inertial> -->
         <visual>
-            <origin xyz="${L2/2} 0 0" rpy="${pi/2} 0 ${pi/2}" />
+            <origin xyz="0 0 0" rpy="0 0 0" />
             <geometry>
                 <box size="${L} ${W} ${H}"/>
@@ -68,29 +68,22 @@
             </material>
         </visual>
-x
-        <collision>
+        <!-- <collision>
             <origin xyz="0 0 0" rpy="0 0 0"/>
             <geometry>
                 <box size="${L} ${W} ${H}"/>
             </geometry>
-        </collision>
+        </collision> -->
     </link>
-    <joint name="joint1" type="continuous">
-        <parent link="base_link" />
-        <child link="arm1" />
-        <origin xyz="0 0 0" rpy="0 0 0"/>
-        <axis xyz="0 0 1"/>
+    <joint name="jointR" type="continuous">
+        <parent link="body" />
+        <child link="rightWheel" />
+        <origin xyz="${L} 0 0" rpy="0 0 0"/>
+        <axis xyz="0 1 0"/>
     </joint>
-    <joint name="joint2" type="continuous">
-        <origin xyz="${L1} 0 0" rpy="0 0 0" />
-        <parent link="arm1" />
-        <child link="arm2" />
-        <axis xyz="0 0 1"/>
-    </joint>
-    <joint name="joint3" type="fixed">
-        <origin xyz="${L2} 0 0" rpy="0 0 0" />
-        <parent link="arm2" />
-        <child link="end_effector" />
-        <axis xyz="0 0 1"/>
+    <joint name="jointL" type="continuous">
+        <origin xyz="${L} 0 0" rpy="0 0 0" />
+        <parent link="bro" />
+        <child link="leftWheel" />
+        <axis xyz="0 1 0"/>
     </joint>
 </robot>
