Commit message: made packages for diff_Drive and arm_move

File: diff_drive/urdf/ddrive.urdf.xacro (robot description, xacro)
@@ -1,5 +1,5 @@
 <?xml version="1.0"?>
 <robot xmlns:xacro="http://wiki.ros.org/wiki/xacro" name="ddrive">
-    <xacro:property name="ddrive" value="$(find homework3)/config/ddrive.yaml"/>
+    <xacro:property name="ddrive" value="$(find diff_drive)/config/ddrive.yaml"/>
     <xacro:property name="ddrive" value="${load_yaml(ddrive)}"/>
     <xacro:property name="wheelW" value="${ddrive['wheelWidth']}"/>

Commit message: made some changes to the launchfile to debug

File: diff_drive/urdf/ddrive.urdf.xacro (robot description, xacro)
@@ -2,10 +2,10 @@
 <robot xmlns:xacro="http://wiki.ros.org/wiki/xacro" name="ddrive">
     <xacro:property name="ddrive" value="$(find diff_drive)/config/ddrive.yaml"/>
-    <xacro:property name="ddrive" value="${load_yaml(ddrive)}"/>
-    <xacro:property name="wheelW" value="${ddrive['wheelWidth']}"/>
-    <xacro:property name="wheelR" value="${ddrive['wheelRadius']}"/>
-    <xacro:property name="L" value="${ddrive['L']}"/>
-    <xacro:property name="W" value="${ddrive['W']}"/>
-    <xacro:property name="H" value="${ddrive['H']}"/>
+    <xacro:property name="drive" value="${load_yaml(ddrive)}"/>
+    <xacro:property name="wheelW" value="${drive['wheelWidth']}"/>
+    <xacro:property name="wheelR" value="${drive['wheelRadius']}"/>
+    <xacro:property name="L" value="${drive['L']}"/>
+    <xacro:property name="W" value="${drive['W']}"/>
+    <xacro:property name="H" value="${drive['H']}"/>
     <xacro:property name='pi' value="3.14159"/>
     <link name="leftWheel">
@@ -31,5 +31,5 @@
         </collision> -->
     </link>
-    <link name="rightWheel">
+    <!-- <link name="rightWheel"> -->
         <!-- <inertial>
             <origin xyz="0 0 0" rpy="0 0 0" />
@@ -37,5 +37,5 @@
             <inertia ixx="${(L2*L2/12) + (R2*R2/4)}"  ixy="0"  ixz="0" iyy="${(L2*L2/12) + (R2*R2/4)}" iyz="0" izz="${(R2*R2/2)}" />
         </inertial> -->
-        <visual>
+        <!-- <visual>
             <origin xyz="${W/2} ${L/2} ${H/2}" rpy="${pi/2} 0 ${pi/2}" />
             <geometry>
@@ -45,5 +45,5 @@
                 <color rgba="1 0 0 1" />
             </material>
-        </visual>
+        </visual> -->
         <!-- <collision>
             <origin xyz="0 0 0" rpy="0 0 0"/>
@@ -52,6 +52,6 @@
             </geometry>
         </collision> -->
-    </link>
-    <link name="body">
+    <!-- </link> -->
+    <!-- <link name="body"> -->
         <!-- <inertial>
             <origin xyz="0 0 0" rpy="0 0 0" />
@@ -59,5 +59,5 @@
             <inertia ixx="${(L2*L2/12) + (R2*R2/4)}"  ixy="0"  ixz="0" iyy="${(L2*L2/12) + (R2*R2/4)}" iyz="0" izz="${(R2*R2/2)}" />
         </inertial> -->
-        <visual>
+        <!-- <visual>
             <origin xyz="0 0 0" rpy="0 0 0" />
             <geometry>
@@ -67,5 +67,5 @@
                 <color rgba="1 0 0 1" />
             </material>
-        </visual>
+        </visual> -->
         <!-- <collision>
             <origin xyz="0 0 0" rpy="0 0 0"/>
@@ -74,6 +74,6 @@
             </geometry>
         </collision> -->
-    </link>
-    <joint name="jointR" type="continuous">
+    <!-- </link> -->
+    <!-- <joint name="jointR" type="continuous">
         <parent link="body" />
         <child link="rightWheel" />
@@ -86,4 +86,4 @@
         <child link="leftWheel" />
         <axis xyz="0 1 0"/>
-    </joint>
+    </joint> -->
 </robot>

Commit message: fixed launchfile error, robot model now loads in rviz with some additional TF errors

File: diff_drive/urdf/ddrive.urdf.xacro (robot description, xacro)
@@ -31,5 +31,5 @@
         </collision> -->
     </link>
-    <!-- <link name="rightWheel"> -->
+    <link name="rightWheel">
         <!-- <inertial>
             <origin xyz="0 0 0" rpy="0 0 0" />
@@ -37,5 +37,5 @@
             <inertia ixx="${(L2*L2/12) + (R2*R2/4)}"  ixy="0"  ixz="0" iyy="${(L2*L2/12) + (R2*R2/4)}" iyz="0" izz="${(R2*R2/2)}" />
         </inertial> -->
-        <!-- <visual>
+        <visual>
             <origin xyz="${W/2} ${L/2} ${H/2}" rpy="${pi/2} 0 ${pi/2}" />
             <geometry>
@@ -45,5 +45,5 @@
                 <color rgba="1 0 0 1" />
             </material>
-        </visual> -->
+        </visual>
         <!-- <collision>
             <origin xyz="0 0 0" rpy="0 0 0"/>
@@ -52,6 +52,6 @@
             </geometry>
         </collision> -->
-    <!-- </link> -->
-    <!-- <link name="body"> -->
+    </link>
+    <link name="body">
         <!-- <inertial>
             <origin xyz="0 0 0" rpy="0 0 0" />
@@ -59,5 +59,5 @@
             <inertia ixx="${(L2*L2/12) + (R2*R2/4)}"  ixy="0"  ixz="0" iyy="${(L2*L2/12) + (R2*R2/4)}" iyz="0" izz="${(R2*R2/2)}" />
         </inertial> -->
-        <!-- <visual>
+        <visual>
             <origin xyz="0 0 0" rpy="0 0 0" />
             <geometry>
@@ -67,5 +67,5 @@
                 <color rgba="1 0 0 1" />
             </material>
-        </visual> -->
+        </visual>
         <!-- <collision>
             <origin xyz="0 0 0" rpy="0 0 0"/>
@@ -74,6 +74,6 @@
             </geometry>
         </collision> -->
-    <!-- </link> -->
-    <!-- <joint name="jointR" type="continuous">
+    </link>
+    <joint name="jointR" type="continuous">
         <parent link="body" />
         <child link="rightWheel" />
@@ -83,7 +83,7 @@
     <joint name="jointL" type="continuous">
         <origin xyz="${L} 0 0" rpy="0 0 0" />
-        <parent link="bro" />
+        <parent link="body" />
         <child link="leftWheel" />
         <axis xyz="0 1 0"/>
-    </joint> -->
+    </joint>
 </robot>

Commit message: made the xacro file display correctly in rviz

File: diff_drive/urdf/ddrive.urdf.xacro (robot description, xacro)
@@ -16,5 +16,5 @@
         </inertial> -->
         <visual>
-            <origin xyz="${-W/2} ${-L/2} ${-H/2}" rpy="${pi/2} 0 ${pi/2}" />
+            <origin xyz="0 0 0" rpy="${pi/2} 0 0" />
             <geometry>
                 <cylinder radius="${wheelR}" length="${wheelW}" />
@@ -24,10 +24,10 @@
             </material>
         </visual>
-        <!-- <collision>
+        <collision>
             <origin xyz="0 0 0" rpy="0 0 0"/>
             <geometry>
                 <cylinder radius="${wheelR}" length="${wheelW}" />
             </geometry>
-        </collision> -->
+        </collision>
     </link>
     <link name="rightWheel">
@@ -38,5 +38,5 @@
         </inertial> -->
         <visual>
-            <origin xyz="${W/2} ${L/2} ${H/2}" rpy="${pi/2} 0 ${pi/2}" />
+            <origin xyz="0 0 0" rpy="${pi/2} 0 0" />
             <geometry>
                 <cylinder radius="${wheelR}" length="${wheelW}" />
@@ -46,10 +46,10 @@
             </material>
         </visual>
-        <!-- <collision>
+        <collision>
             <origin xyz="0 0 0" rpy="0 0 0"/>
             <geometry>
                 <cylinder radius="${wheelR}" length="${wheelW}" />
             </geometry>
-        </collision> -->
+        </collision>
     </link>
     <link name="body">
@@ -68,19 +68,21 @@
             </material>
         </visual>
-        <!-- <collision>
+        <collision>
             <origin xyz="0 0 0" rpy="0 0 0"/>
             <geometry>
                 <box size="${L} ${W} ${H}"/>
             </geometry>
-        </collision> -->
+        </collision>
     </link>
+<!-- red wheel -->
     <joint name="jointR" type="continuous">
         <parent link="body" />
         <child link="rightWheel" />
-        <origin xyz="${L} 0 0" rpy="0 0 0"/>
+        <origin xyz="${-L/2} ${W/2} 0" rpy="0 0 0"/>
         <axis xyz="0 1 0"/>
     </joint>
+<!-- blue wheel -->
     <joint name="jointL" type="continuous">
-        <origin xyz="${L} 0 0" rpy="0 0 0" />
+        <origin xyz="${-L/2} ${-W/2} 0" rpy="0 0 0" />
         <parent link="body" />
         <child link="leftWheel" />

Commit message: finished xacro, starting gazebo xacro

File: diff_drive/urdf/ddrive.urdf.xacro (robot description, xacro)
@@ -5,4 +5,6 @@
     <xacro:property name="wheelW" value="${drive['wheelWidth']}"/>
     <xacro:property name="wheelR" value="${drive['wheelRadius']}"/>
+    <xacro:property name="tW" value="${drive['topWheelWidth']}"/>
+    <xacro:property name="tR" value="${drive['topWheelRadius']}"/>
     <xacro:property name="L" value="${drive['L']}"/>
     <xacro:property name="W" value="${drive['W']}"/>
@@ -75,17 +77,75 @@
         </collision>
     </link>
+    <link name="topWheel">
+        <!-- <inertial>
+            <origin xyz="0 0 0" rpy="0 0 0" />
+            <mass value="1"/>
+            <inertia ixx="${(L2*L2/12) + (R2*R2/4)}"  ixy="0"  ixz="0" iyy="${(L2*L2/12) + (R2*R2/4)}" iyz="0" izz="${(R2*R2/2)}" />
+        </inertial> -->
+        <visual>
+            <origin xyz="0 0 0" rpy="${pi/2} 0 0" />
+            <geometry>
+                <cylinder radius="${tR}" length="${tW}" />
+            </geometry>
+            <material name="red_mat">
+                <color rgba="1 0 0 1" />
+            </material>
+        </visual>
+        <collision>
+            <origin xyz="0 0 0" rpy="0 0 0"/>
+            <geometry>
+                <cylinder radius="${tR}" length="${tW}" />
+            </geometry>
+        </collision>
+    </link>
+    <link name="botWheel">
+        <!-- <inertial>
+            <origin xyz="0 0 0" rpy="0 0 0" />
+            <mass value="1"/>
+            <inertia ixx="${(L2*L2/12) + (R2*R2/4)}"  ixy="0"  ixz="0" iyy="${(L2*L2/12) + (R2*R2/4)}" iyz="0" izz="${(R2*R2/2)}" />
+        </inertial> -->
+        <visual>
+            <origin xyz="0 0 0" rpy="${pi/2} 0 0" />
+            <geometry>
+                <cylinder radius="${tR}" length="${tW}" />
+            </geometry>
+            <material name="green_mat">
+                <color rgba="0 1 0 1" />
+            </material>
+        </visual>
+        <collision>
+            <origin xyz="0 0 0" rpy="0 0 0"/>
+            <geometry>
+                <cylinder radius="${tR}" length="${tW}" />
+            </geometry>
+        </collision>
+    </link>
 <!-- red wheel -->
     <joint name="jointR" type="continuous">
         <parent link="body" />
         <child link="rightWheel" />
-        <origin xyz="${-L/2} ${W/2} 0" rpy="0 0 0"/>
+        <origin xyz="${-wheelR/2} ${(W/2)+wheelW/2} 0" rpy="0 0 0"/>
         <axis xyz="0 1 0"/>
     </joint>
 <!-- blue wheel -->
     <joint name="jointL" type="continuous">
-        <origin xyz="${-L/2} ${-W/2} 0" rpy="0 0 0" />
+        <origin xyz="${-wheelR/2} ${(-W/2)-wheelW/2} 0" rpy="0 0 0" />
         <parent link="body" />
         <child link="leftWheel" />
         <axis xyz="0 1 0"/>
     </joint>
+<!-- top wheel -->
+    <joint name="jointT" type="fixed">
+        <origin xyz="${L/2} 0 ${tR}" rpy="0 0 0" />
+        <parent link="body" />
+        <child link="topWheel" />
+        <axis xyz="0 1 0"/>
+    </joint>
+<!-- bottom wheel -->
+    <joint name="jointB" type="continuous">
+        <origin xyz="${L/2} 0 ${-tR}" rpy="0 0 0" />
+        <parent link="body" />
+        <child link="botWheel" />
+        <axis xyz="0 1 0"/>
+    </joint>
 </robot>

Commit message: Robot displays in gazebo using launchfile

File: diff_drive/urdf/ddrive.urdf.xacro (robot description, xacro)
@@ -11,11 +11,12 @@
     <xacro:property name="H" value="${drive['H']}"/>
     <xacro:property name='pi' value="3.14159"/>
-    <xacro:include filename="$(find diff_drive)/urdf/ddrive.gazebo.xacro"/>
+    <!-- <xacro:include filename="$(find diff_drive)/urdf/ddrive.gazebo.xacro"/> -->
+    <link name="base_link"/>
     <link name="leftWheel">
-        <!-- <inertial>
+        <inertial>
             <origin xyz="0 0 0" rpy="0 0 0" />
-            <mass value="1"/>
-            <inertia ixx="${(L1*L1/12) + (R1*R1/4)}"  ixy="0"  ixz="0" iyy="${(L1*L1/12) + (R1*R1/4)}" iyz="0" izz="${(R1*R1/2)}" />
-        </inertial> -->
+            <mass value="0.5"/>
+            <inertia ixx="${1/12*(3*wheelR*wheelR + wheelW*wheelW)}"  ixy="0"  ixz="0" iyy="${1/12*wheelR*wheelR}" iyz="0" izz="${1/12*(3*wheelR*wheelR + wheelW*wheelW)}" />
+        </inertial>
         <visual>
             <origin xyz="0 0 0" rpy="${pi/2} 0 0" />
@@ -35,9 +36,9 @@
     </link>
     <link name="rightWheel">
-        <!-- <inertial>
+        <inertial>
             <origin xyz="0 0 0" rpy="0 0 0" />
-            <mass value="1"/>
-            <inertia ixx="${(L2*L2/12) + (R2*R2/4)}"  ixy="0"  ixz="0" iyy="${(L2*L2/12) + (R2*R2/4)}" iyz="0" izz="${(R2*R2/2)}" />
-        </inertial> -->
+            <mass value="0.5"/>
+            <inertia ixx="${1/12*(3*wheelR*wheelR + wheelW*wheelW)}"  ixy="0"  ixz="0" iyy="${1/12*wheelR*wheelR}" iyz="0" izz="${1/12*(3*wheelR*wheelR + wheelW*wheelW)}" />
+        </inertial>
         <visual>
             <origin xyz="0 0 0" rpy="${pi/2} 0 0" />
@@ -57,9 +58,9 @@
     </link>
     <link name="body">
-        <!-- <inertial>
+        <inertial>
             <origin xyz="0 0 0" rpy="0 0 0" />
-            <mass value="1"/>
-            <inertia ixx="${(L2*L2/12) + (R2*R2/4)}"  ixy="0"  ixz="0" iyy="${(L2*L2/12) + (R2*R2/4)}" iyz="0" izz="${(R2*R2/2)}" />
-        </inertial> -->
+            <mass value="2"/>
+            <inertia ixx="${1/12*(W*W + H*H)}"  ixy="0"  ixz="0" iyy="${1/12*(W*W+L*L)}" iyz="0" izz="${1/12*(H*H+L*L)}"/>
+        </inertial>
         <visual>
             <origin xyz="0 0 0" rpy="0 0 0" />
@@ -79,9 +80,9 @@
     </link>
     <link name="topWheel">
-        <!-- <inertial>
+        <inertial>
             <origin xyz="0 0 0" rpy="0 0 0" />
-            <mass value="1"/>
-            <inertia ixx="${(L2*L2/12) + (R2*R2/4)}"  ixy="0"  ixz="0" iyy="${(L2*L2/12) + (R2*R2/4)}" iyz="0" izz="${(R2*R2/2)}" />
-        </inertial> -->
+            <mass value="0.25"/>
+            <inertia ixx="${1/12*(3*tR*tR + tW*tW)}"  ixy="0"  ixz="0" iyy="${1/12*tR*tR}" iyz="0" izz="${1/12*(3*tR*tR + tW*tW)}" />
+        </inertial>
         <visual>
             <origin xyz="0 0 0" rpy="${pi/2} 0 0" />
@@ -101,9 +102,9 @@
     </link>
     <link name="botWheel">
-        <!-- <inertial>
+        <inertial>
             <origin xyz="0 0 0" rpy="0 0 0" />
-            <mass value="1"/>
-            <inertia ixx="${(L2*L2/12) + (R2*R2/4)}"  ixy="0"  ixz="0" iyy="${(L2*L2/12) + (R2*R2/4)}" iyz="0" izz="${(R2*R2/2)}" />
-        </inertial> -->
+            <mass value="0.25"/>
+            <inertia ixx="${1/12*(3*tR*tR + tW*tW)}"  ixy="0"  ixz="0" iyy="${1/12*tR*tR}" iyz="0" izz="${1/12*(3*tR*tR + tW*tW)}" />
+        </inertial>
         <visual>
             <origin xyz="0 0 0" rpy="${pi/2} 0 0" />
@@ -122,4 +123,10 @@
         </collision>
     </link>
+    <joint name="joint1" type="fixed">
+        <parent link="base_link" />
+        <child link="body" />
+        <origin xyz="0 0 0" rpy="0 0 0"/>
+        <axis xyz="0 0 0"/>
+    </joint>
 <!-- red wheel -->
     <joint name="jointR" type="continuous">

Commit message: Made the robot move for some time

File: diff_drive/urdf/ddrive.urdf.xacro (robot description, xacro)
@@ -16,5 +16,5 @@
         <inertial>
             <origin xyz="0 0 0" rpy="0 0 0" />
-            <mass value="0.5"/>
+            <mass value="2"/>
             <inertia ixx="${1/12*(3*wheelR*wheelR + wheelW*wheelW)}"  ixy="0"  ixz="0" iyy="${1/12*wheelR*wheelR}" iyz="0" izz="${1/12*(3*wheelR*wheelR + wheelW*wheelW)}" />
         </inertial>
@@ -29,5 +29,5 @@
         </visual>
         <collision>
-            <origin xyz="0 0 0" rpy="0 0 0"/>
+            <origin xyz="0 0 0" rpy="${pi/2} 0 0"/>
             <geometry>
                 <cylinder radius="${wheelR}" length="${wheelW}" />
@@ -38,5 +38,5 @@
         <inertial>
             <origin xyz="0 0 0" rpy="0 0 0" />
-            <mass value="0.5"/>
+            <mass value="2"/>
             <inertia ixx="${1/12*(3*wheelR*wheelR + wheelW*wheelW)}"  ixy="0"  ixz="0" iyy="${1/12*wheelR*wheelR}" iyz="0" izz="${1/12*(3*wheelR*wheelR + wheelW*wheelW)}" />
         </inertial>
@@ -51,5 +51,5 @@
         </visual>
         <collision>
-            <origin xyz="0 0 0" rpy="0 0 0"/>
+            <origin xyz="0 0 0" rpy="${pi/2} 0 0"/>
             <geometry>
                 <cylinder radius="${wheelR}" length="${wheelW}" />
@@ -60,5 +60,5 @@
         <inertial>
             <origin xyz="0 0 0" rpy="0 0 0" />
-            <mass value="2"/>
+            <mass value="1"/>
             <inertia ixx="${1/12*(W*W + H*H)}"  ixy="0"  ixz="0" iyy="${1/12*(W*W+L*L)}" iyz="0" izz="${1/12*(H*H+L*L)}"/>
         </inertial>
@@ -95,5 +95,5 @@
         </visual>
         <collision>
-            <origin xyz="0 0 0" rpy="0 0 0"/>
+            <origin xyz="0 0 0" rpy="${pi/2} 0 0"/>
             <geometry>
                 <cylinder radius="${tR}" length="${tW}" />
@@ -117,5 +117,5 @@
         </visual>
         <collision>
-            <origin xyz="0 0 0" rpy="0 0 0"/>
+            <origin xyz="0 0 0" rpy="${pi/2} 0 0"/>
             <geometry>
                 <cylinder radius="${tR}" length="${tW}" />

Commit message: took video of diff drive robot flipping

File: diff_drive/urdf/ddrive.urdf.xacro (robot description, xacro)
@@ -16,5 +16,5 @@
         <inertial>
             <origin xyz="0 0 0" rpy="0 0 0" />
-            <mass value="2"/>
+            <mass value="10"/>
             <inertia ixx="${1/12*(3*wheelR*wheelR + wheelW*wheelW)}"  ixy="0"  ixz="0" iyy="${1/12*wheelR*wheelR}" iyz="0" izz="${1/12*(3*wheelR*wheelR + wheelW*wheelW)}" />
         </inertial>
@@ -38,5 +38,5 @@
         <inertial>
             <origin xyz="0 0 0" rpy="0 0 0" />
-            <mass value="2"/>
+            <mass value="10"/>
             <inertia ixx="${1/12*(3*wheelR*wheelR + wheelW*wheelW)}"  ixy="0"  ixz="0" iyy="${1/12*wheelR*wheelR}" iyz="0" izz="${1/12*(3*wheelR*wheelR + wheelW*wheelW)}" />
         </inertial>
